File: myth.kicad_sch (KiCad schematic)
At the start: 143 parts, among them J1 Conn_01x08_Male, J2 Conn_01x08_Male, J4 Conn_01x08_Male, J5 Conn_01x08_Male, J6 Conn_01x08_Male, U1 74AHC02, U10 74HC595, U100 74AHC08, U101 74LS32, U102 74LS08, U103 74HC00, U104 74LS08, U105 74AHC02, U106 74LS08, U107 74LS08, U108 74LS08, U109 74LS573, U11 74HC165, U110 74LS573, U111 74HC157, U112 74HC157, U113 74HC157, U114 74AHC08, U115 4002, U116 4072, U117 74LS573, U118 74HC02, U119 74LS573, U12 74AHC08, U120 74LS573, U121 74AHC273, U122 74HC157, U123 74LS32, U124 74AHC04, U125 74LS573, U126 74LS573, U127 74AHC08, U128 74LS27, U129 74HC00, U13 74HC238, U130 74AHC08, U131 74LS573, U132 74HC74, U133 4072, U134 4072, U135 4078, U14 74HC238, U15 74HC238, U16 4002, U17 74AHC273, U18 74LS32, U19 CD4532BE, U2 74AHC04, U20 74AHC138, U21 74AHC04, U22 74AHC138, U23 74HC238, U24 74HC238, U25 74LS32, U27 74AHC244, U28 74HC238, U29 74HC238, U3 74HC74, U30 4075, U31 74AHC04, U32 74HC00, U33 74HC163, U34 74AHC138, U35 74AHC138, U36 74HC238, U37 74AHC138, U38 74LS32, U39 74HC238, U4 74LS11, U40 74AHC02, U41 74AHC574, U42 74LS573, U43 74HC157, U44 74HC157, U45 74HC193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

Commit message: Fix comments in schematics
Parts:
- removed U42: 74LS573, Package_DIP:DIP-16_W7.62mm_Socket_LongPads, symbol 74xx:74LS573
- added U26, U42: 74AHC374, symbol 74xx:74AHC374
Connections:
- net DB0: now also U26.2 (O0)
- net DB1: now also U26.5 (O1)
- net DB2: now also U26.6 (O2)
- net DB3: now also U26.9 (O3)
- net DB4: now also U26.12 (O4)
- net DB5: now also U26.15 (O5)
- net DB6: now also U26.16 (O6)
- net DB7: now also U26.19 (O7)
- net GND: now also U26.10 (GND)
- net IB0: now also U26.3 (D0)
- net IB1: now also U26.4 (D1)
- net IB2: now also U26.7 (D2)
- net IB3: now also U26.8 (D3)
- net IB4: now also U26.13 (D4)
- net IB5: now also U26.14 (D5)
- net IB6: now also U26.17 (D6)
- net IB7: now also U26.18 (D7)
- net SH1_PARLE: now also U26.11 (Cp)
- net VCC: now also U26.20 (VCC)
- net ~{Px}: now also U26.1 (OE)
- no-connect marks 47 -> 46
Other:
- note added: "8 AND ("A boolean-and T") 9 IOR ("A inclusive-or T") 10 EOR ("A exclusive-or T") 11 ADD ("Add T to A) 12 CAR ("Carry bit of: A plus T") 13 ALT ("Is A less than T") 14 AET ("Is A equal to T") 15 AGT ("Is A greater than T")"
- note added: "B: - Saves page index of current instruction byte during call/trap/go - Outputs return page index during RTS - Is the implied page index for memory read-write, with the corresponding byte offset stored in O (Offset) - Together with O forms a 16-bit address pointers subject to the xU instruction The B:O pointer can be loaded from/saved into the BO-Pointers P1-4"
- note added: "B:O Pointer high"
- note added: "B:O Pointer low"
- note added: "IPH: Instruction Fetch Phase DPH: Data Phase"
- note added: "Instruction byte: all0: OPC_SYS 00000 xxx See table @ SYS decoder else: OPC_BOPS 00001 xxx See table @ BOPS decoder OPC_ALU 0001 xxxx See table @ ALU OPC_TRAP 001 xxxxx b0-4: DEST PAGE OPC_GETPUT 01 xx x xxx b0-2 OFFS, b3:GET/PUT, B4-5:REG(GETPUT) OPC_PAIR 1 xxx xxxx b0-3 DST, b4-6 SRC"
- note added: "O: - Saves offset of current instruction byte during call/trap/go - Outputs return offset during RTS - Is the (only!) implied address offset for memory read-write, with the corresponding page index stored in B (Base) - Together with B forms 16-bit address pointers subject to the xU instruction. The B:O pointer can be loaded from/saved into the BO-Pointers P1-4"
- note added: "PHA0: Put page index (C) and byte offset (PC) of instruction on address bus PHA1: Latch opcode or IRQ Trap opcode into IB0-7, pre-decode instruction PHA2: Decode instruction, set up source byte on DB or other action PHA3: Latch results into target registers or other action CLOSE: Finish latching results, reset clock counter"
- note added: "The L register is decremented during CALL/TRAP/ENTER and incremented during RTS/RTI/LEAVE This operations provide single-page local stack frames for nested subroutines. Each local page has "GETPUT" variables called L0-L7 at byte offsets 0xF8-0xFF."
- note removed: "573! Transparent Latch follows input"
- note removed: "8 AND ("A boolean-and T") 9 IOR ("A inclusive-or T") 10 EOR ("A exclusive-or T") 11 ADD ("Add T to A) 12 CAR ("Carry bit of: A plus T") 13 AL_ ("Is A less than T") 14 AE_ ("Is A equal to T") 15 AG_ ("Is A greater than T")"
- note removed: "B: - Saves page index of current instruction byte during call/trap/go - Outputs RTSurn page index during RTS - Is the implied page index for memory read-write, with the corresponding byte offset stored in O (Offset) - Together with O forms a 16-bit address pointers subject to the xU instruction The B:O pointer can be loaded from/saved into the BO-Pointers P1-4"
- note removed: "Instruction byte: all0: OPC_SYS 00000 xxx See table @ SYS decoder else: OPC_STASH 00001 xxx See table @ STASH decoder OPC_ALU 0001 xxxx See table @ ALU OPC_TRAP 001 xxxxx b0-4: DEST PAGE OPC_GETPUT 01 xx x xxx b0-2 OFFS, b3:GET/PUT, B4-5:REG(GETPUT) OPC_PAIR 1 xxx xxxx b0-3 DST, b4-6 SRC"
- note removed: "O: - Saves offset of current instruction byte during call/trap/go - Outputs RTSurn offset during RTS - Is the (only!) implied address offset for memory read-write, with the corresponding page index stored in B (Base) - Together with B forms 16-bit address pointers subject to the xU instruction. The B:O pointer can be loaded from/saved into the BO-Pointers P1-4"
- note removed: "PHA0: Put page index (C) and byte offset (PC) of instruction on address bus PHA1: Latch opcode or IRQ Trap opcode into IB0-7, pre-decode instruction PHA2: Decode instruction, set up source byte on DB or other action PHA3: Latch results into target registers or other action CLOSE: Finish latching etc."
- note removed: "Pointer high"
- note removed: "Pointer low"
- note removed: "The L register is decremented during CALL/TRAP/ENTER and incremented during RTS/LEAVE This operations provide single-page local stack frames for nested subroutines. Each local page has "GETPUT" variables called L0-L7 at byte offsets 0xF8-0xFF."
- moved on the sheet: U102B, U103B, U104B, U106B, U106D, U107B, U111, U118D, U121, U122, U123A, U124A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

Commit message: Reformat IO section
Parts:
- removed U42: 74AHC374, symbol 74xx:74AHC374
Connections:
- net EH0: no longer U23.1 (A0)
- net EH1: no longer U23.2 (A1)
- net EH2: no longer U23.3 (A2)
- net GND: no longer U23.5 (~{G2B})
- net ~{RTS}: now also U106.12, U20.9 (O6); no longer U106.11, U108.13
- net RTS renamed RET
- net SH1_PARLE renamed PLE
- net SL1_PAROE renamed POE
- net ~{SL1_PAROE} renamed ~{POE}
- new net ~{RET}: U106.11, U108.13
Other:
- note added: "B: - Saves page index of current instruction byte during call/trap/go - Outputs return page index during RET - Is the implied page index for memory read-write, with the corresponding byte offset stored in O (Offset) - Together with O forms a 16-bit address pointers subject to the xU instruction The B:O pointer can be loaded from/saved into the BO-Pointers P1-4"
- note added: "Device Enable Register"
- note added: "External GPIO BUS"
- note added: "O: - Saves offset of current instruction byte during call/trap/go - Outputs return offset during RET - Is the (only!) implied address offset for memory read-write, with the corresponding page index stored in B (Base) - Together with B forms 16-bit address pointers subject to the xU instruction. The B:O pointer can be loaded from/saved into the BO-Pointers P1-4"
- note added: "On RET/xG/xC: Load instruction offset from O into PC"
- note added: "On RET: Restore PC value from O register (Center right)"
- note added: "Parallel Input Register"
- note added: "Parallel LE"
- note added: "Parallel OE"
- note added: "Parallel Output Register"
- note added: "Register at CLOSE xU instruction adder would feedback B0-7 goes to PC module latched during RET"
- note added: "Serial Input Register"
- note added: "Serial Output Register"
- note added: "The L register is decremented during CALL/TRAP/ENTER and incremented during RET/LEAVE This operations provide single-page local stack frames for nested subroutines. Each local page has "GETPUT" variables called L0-L7 at byte offsets 0xF8-0xFF."
- note removed: "8-bit GPIO"
- note removed: "B: - Saves page index of current instruction byte during call/trap/go - Outputs return page index during RTS - Is the implied page index for memory read-write, with the corresponding byte offset stored in O (Offset) - Together with O forms a 16-bit address pointers subject to the xU instruction The B:O pointer can be loaded from/saved into the BO-Pointers P1-4"
- note removed: "Device Enable"
- note removed: "O: - Saves offset of current instruction byte during call/trap/go - Outputs return offset during RTS - Is the (only!) implied address offset for memory read-write, with the corresponding page index stored in B (Base) - Together with B forms 16-bit address pointers subject to the xU instruction. The B:O pointer can be loaded from/saved into the BO-Pointers P1-4"
- note removed: "On RTS/xG/xC: Load instruction offset from O into PC"
- note removed: "On RTS: Restore PC value from O register (Center right)"
- note removed: "Register at CLOSE xU instruction adder would feedback B0-7 goes to PC module latched during RTS"
- note removed: "The L register is decremented during CALL/TRAP/ENTER and incremented during RTS/RTI/LEAVE This operations provide single-page local stack frames for nested subroutines. Each local page has "GETPUT" variables called L0-L7 at byte offsets 0xF8-0xFF."
- moved on the sheet: R1, RN1, RN2, U10, U11, U17, U1D, U23, U24, U26, U28, U29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
