File: myth.kicad_sch (KiCad schematic)
At the start: 151 parts, among them J1 Conn_01x08_Male, J2 Conn_01x08_Male, J4 Conn_01x08_Male, J5 Conn_01x08_Male, J6 Conn_01x08_Male, U1 74AHC02, U10 74HC595, U100 74AHC08, U101 74LS32, U102 74LS08, U103 74HC00, U104 74LS08, U105 74AHC02, U106 74LS08, U107 74LS08, U108 74LS08, U109 74LS573, U11 74HC165, U110 74LS573, U111 74HC157, U112 74HC157, U113 74HC157, U114 74AHC08, U115 4002, U116 4072, U117 74LS573, U118 74LS32, U119 74LS573, U12 74AHC08, U120 74LS573, U121 74AHC273, U122 74HC157, U123 74LS32, U124 74AHC04, U125 74LS573, U126 74LS573, U127 74AHC08, U128 74LS27, U129 74HC00, U13 74HC238, U130 74AHC08, U131 74LS573, U132 74HC74, U133 4072, U134 4072, U135 4078, U136 74AHC244, U137 74LS32, U138 74LS32, U139 74AHC273, U14 74HC238, U140 74LS32, U141 74LS32, U142 74AHC04, U144 74LS32, U15 74HC238, U16 4002, U17 74AHC273, U19 CD4532BE, U2 74AHC04, U20 74AHC138, U21 74AHC04, U22 74AHC138, U23 74HC238, U24 74HC238, U25 74LS32, U26 74AHC374, U27 74AHC244, U28 74HC238, U29 74HC238, U3 74HC74, U30 4075, U31 74AHC04, U32 74HC00, U33 74HC163, U34 74AHC138, U35 74AHC138, U36 74HC238, U37 74AHC138, U38 74LS32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

Commit message: Reorder regs, change xR instruction, update docs
Parts:
- removed U16: 4002, Package_DIP:DIP-14_W7.62mm_Socket_LongPads, symbol 4xxx:4002
- removed U84: 74AHC273, Package_DIP:DIP-20_W7.62mm_Socket_LongPads, symbol 74xx:74HC273
- added U143: 74AHC374, symbol 74xx:74AHC374
- added U145: 4078, symbol 4xxx_IEEE:4078
- added U84: 74AHC244, Package_DIP:DIP-20_W7.62mm_Socket_LongPads, symbol 74xx:74AHC244
Connections:
- net CLOSE: now also U143.11 (Cp)
- net GND: now also U143.10 (GND), U145.10, U145.11, U145.7 (Vss), U145.9, U84.10 (GND), U84.13 (2A2), U84.15 (2A1), U84.17 (2A0), U84.2 (1A0), U84.4 (1A1), U84.6 (1A2), U84.8 (1A3)
- net O0: now also U143.3 (D0)
- net O0_old: now also U143.2 (O0), U84.18 (1Y0)
- net O1: now also U143.4 (D1)
- net O1_old: now also U143.5 (O1), U84.16 (1Y1)
- net O2: now also U143.7 (D2)
- net O2_old: now also U143.6 (O2), U84.14 (1Y2)
- net O3: now also U143.8 (D3)
- net O3_old: now also U143.9 (O3), U84.12 (1Y3)
- net O4: now also U143.13 (D4)
- net O4_old: now also U143.12 (O4), U84.3 (2Y0)
- net O5: now also U143.14 (D5)
- net O5_old: now also U143.15 (O5), U84.5 (2Y1)
- net O6: now also U143.17 (D6)
- net O6_old: now also U143.16 (O6), U84.7 (2Y2)
- net O7: now also U143.18 (D7)
- net O7_old: now also U143.19 (O7), U84.9 (2Y3)
- net VCC: now also U143.20 (VCC), U145.14 (Vdd), U84.11 (2A3), U84.20 (VCC)
- net xH: now also U36.12 (Y3); no longer U36.11 (Y4)
- net xJ: now also U145.3
- net xN: now also U36.10 (Y5); no longer U36.9 (Y6)
- net xR: now also U36.9 (Y6), U143.1 (OE), U145.12
- net xU: no longer U36.14 (Y1)
- net xW: now also U36.14 (Y1); no longer U36.12 (Y3)
- net xZ: now also U36.11 (Y4); no longer U36.10 (Y5)
- net ~{JUMP}: now also U145.13
- net ~{xR}: now also U84.1 (1OE), U84.19 (2OE); no longer U37.15 (O0)
- net at U7.8: now also U145.2
- net at U7.6: now also U145.4
- net at U38.6: now also U145.5
- new net ~{xU}: U37.15 (O0)
- no-connect marks 43 -> 44
Other:
- note added: "8 AND ("A boolean-and X") 9 IOR ("A inclusive-or X") 10 EOR ("A exclusive-or X") 11 ADD ("Add X to A) 12 OVF ("Overflow bits of: A+B") 13 ALX ("A less than X") 14 AEX ("A equal to X") 15 AGX ("A greater than X")"
- note added: "A := A & X A := A | X A := A ^ X A := A + X, bits 0-7 A := Zero + B6:V + B7:CARRY A := (A<X)? FFh:0 A := (A==X)? FFh:0 A := (A>X)? FFh:0"
- note added: "OE except when xR"
- note added: "OE when xR"
- note added: "Outputs hardwired offset 80h"
- note added: "Register at CLOSE to avoid xU adder feedback Registered byte goes to PC module, latched during RET"
- note added: "xR: sets page, branch to fixed offset 80h"
- note removed: "8 AND ("A boolean-and X") 9 IOR ("A inclusive-or X") 10 EOR ("A exclusive-or X") 11 ADD ("Add X to A) 12 OVF ("Carry/Overflow of: A plus X") 13 ALX ("A less than X") 14 AEX ("A equal to X") 15 AGX ("A greater than X")"
- note removed: "A := A & X A := A | X A := A ^ X A := A + X, bits 0-7 A := Zero + LSB=CARRY + MSB=OVERFLOW bit of: A+X A := (A<X)? FFh:0 A := (A==X)? FFh:0 A := (A>X)? FFh:0"
- note removed: "Register at CLOSE xU instruction adder would feedback B0-7 goes to PC module latched during RET"
- moved on the sheet: J1, J2, J4, J5, J6, U100D, U102B, U103B, U104B, U105A, U106B, U106D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

Commit message: Fix bug in schematics
Parts:
- added U146: 74AHC08, Package_DIP:DIP-14_W7.62mm_Socket_LongPads, symbol 74xx:74LS08
Connections:
- net JUMP: now also U146.12; no longer U43.1 (S)
- net ~{xR}: now also U146.13
- new net: U146.11, U43.1 (S)
Changed lines of the file:
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@@
 	(text "On RET:\nRestore PC value\nfrom O register\n(Center right)"
 		(exclude_from_sim no)
-		(at 486.664 376.174 0)
+		(at 491.744 379.222 0)
 		(effects
 			(font
@@
 	(wire
 		(pts
+			(xy 499.11 358.14) (xy 515.62 358.14)
+		)
+		(stroke
+			(width 0)
+			(type default)
+		)
+	)
+	(wire
+		(pts
 			(xy 806.45 748.03) (xy 825.5 748.03)
 		)
@@
 		)
 	)
+	(label "~{xR}"
+		(at 483.87 360.68 180)
+		(effects
+			(font
+				(size 1.27 1.27)
+			)
+			(justify right bottom)
+		)
+	)
 	(label "LL0"
 		(at 665.48 676.91 180)
@@
 	)
 	(label "JUMP"
-		(at 515.62 358.14 180)
+		(at 483.87 355.6 180)
 		(effects
 			(font
@@
 				)
 			)
+		)
+	)
+	(symbol
+		(lib_id "74xx:74LS08")
+		(at 491.49 358.14 0)
+		(unit 4)
+		(exclude_from_sim no)
+		(in_bom yes)
+		(on_board yes)
+		(dnp no)
+		(property "Reference" "U146"
+			(at 491.49 349.885 0)
+			(effects
+				(font
+					(size 1.27 1.27)
+				)
+			)
+		)
+		(property "Value" "74AHC08"
+			(at 491.49 352.1964 0)
+			(effects
+				(font
+					(size 1.27 1.27)
+				)
+			)
+		)
+		(property "Footprint" "Package_DIP:DIP-14_W7.62mm_Socket_LongPads"
+			(at 491.49 358.14 0)
+			(effects
+				(font
+					(size 1.27 1.27)
+				)
+				(hide yes)
+			)
+		)
+		(property "Datasheet" "http://www.ti.com/lit/gpn/sn74LS08"
+			(at 491.49 358.14 0)
+			(effects
+				(font
+					(size 1.27 1.27)
+				)
+				(hide yes)
+			)
+		)
+		(property "Description" ""
+			(at 491.49 358.14 0)
+			(effects
+				(font
+					(size 1.27 1.27)
+				)
+				(hide yes)
+			)
+		)
+		(pin "1"
+		)
+		(pin "2"
+		)
+		(pin "3"
+		)
+		(pin "4"
+		)
+		(pin "5"
+		)
+		(pin "6"
+		)
+		(pin "10"
+		)
+		(pin "8"
+		)
+		(pin "9"
+		)
+		(pin "11"
+		)
+		(pin "12"
+		)
+		(pin "13"
+		)
+		(pin "14"
+		)
+		(pin "7"
+		)
+		(instances
+			(project "myth"
+				(path "/29cbb0bc-f66b-4d11-80e7-5bb270e42496"
+					(reference "U146")
+					(unit 4)
+				)
+			)
